File: hardware/holter_monitor.kicad_pcb (KiCad board)
At the start: 2 copper layers, 52 parts, among them J1 USB_C_Receptacle_USB2.0_16P, J2 BAT JST-PH, J3 AD8232, J4 UART, Q1 AO3401A, SW1 SW_SPDT, SW2 RESET, SW3 BOOT, U1 USBLC6-2SC6, U2 MCP73831-2-OT, U3 AP2112K-3.3, U4 ESP32-S3-WROOM-1

Commit message: Switched from AD8232 footprint to complete SEN-12650 module footprint
Parts:
- moved C10 124.6 mm to (62.2, 185.8)
- moved C11 124.6 mm to (62.2, 188.8)
- moved C7 124.6 mm to (62.2, 176.7)
- moved C8 124.6 mm to (62.2, 179.8)
- moved J2 124.6 mm to (70.8, 167.2)
- moved R1 124.6 mm to (21.1, 176.7)
- moved R10 124.6 mm to (25.9, 185.6)
- moved R12 124.6 mm to (25.9, 191.5)
- moved R13 124.6 mm to (30.6, 176.7)
- moved R14 124.6 mm to (30.6, 179.7)
- moved R15 124.6 mm to (30.6, 182.6)
- moved R2 124.6 mm to (21.1, 179.7)
- moved R3 124.6 mm to (21.1, 182.6)
- moved R4 124.6 mm to (21.1, 185.6)
- moved R6 124.6 mm to (21.1, 191.5)
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Other:
- board outline added: 70 x 90 mm

Commit message: Added switches, uart and battery pins to the pcb design
Parts:
- removed J3: AD8232, Connector_PinSocket_2.54mm:PinSocket_1x06_P2.54mm_Vertical
- added U5: SEN-12650, SEN-12650:MODULE_SEN-12650, F.Cu at (143.6, 133.8)
- moved SW1 154.9 mm to (180.5, 120.5), turned to -90 degrees
- moved J4 125.0 mm to (183.0, 67.5)
- moved J2 105.2 mm to (171.5, 137.0)
- moved SW3 104.2 mm to (163.0, 140.0)
- moved SW2 77.5 mm to (136.5, 140.0)
- moved U4 16.0 mm to (150.0, 66.0)
- moved J1 0.30 mm to (150.0, 140.3)

Commit message: Placed all of the elements on the board
Parts:
- moved R7 168.8 mm to (162.3, 77.3), turned to 180 degrees
- moved R6 168.3 mm to (132.2, 65.0), turned to 180 degrees
- moved R5 168.3 mm to (173.2, 116.4), turned to 180 degrees
- moved R8 166.2 mm to (160.3, 82.0)
- moved TP4 163.1 mm to (171.3, 87.0)
- moved R12 162.6 mm to (150.6, 87.1)
- moved R3 161.3 mm to (170.6, 121.8), turned to 90 degrees
- moved R11 157.0 mm to (145.6, 87.0)
- moved R9 156.1 mm to (132.6, 68.7), turned to 180 degrees
- moved R4 154.4 mm to (164.7, 128.9)
- moved R13 153.9 mm to (155.7, 87.1)
- moved C6 152.9 mm to (137.6, 61.5), turned to 90 degrees
- moved R10 151.4 mm to (140.8, 87.0)
- moved TP2 148.4 mm to (180.2, 120.2)
- moved R14 148.3 mm to (135.6, 75.0)
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Connections:
- U4 pad 17: unconnected-(U4-IO9-Pad17) -> VBAT_SENSE
- U4 pad 18: unconnected-(U4-IO10-Pad18) -> VBUS_SENSE
- U4 pad 5: VBAT_SENSE -> unconnected-(U4-IO5-Pad5)
- U4 pad 6: VBUS_SENSE -> unconnected-(U4-IO6-Pad6)
